Commit message: update robot urdf

File: slam/delivery_robot/urdf/delivery_robot.urdf (robot description, URDF)
Before this commit: robot delivery_robot, 4 links, 3 joints
Links:
- removed link laser
- link base_link: mass 5.1663 -> 3.92914679746778
- link left_wheel: mass 0.15849 -> 0.158485151112061
- link right_wheel: mass 0.15849 -> 0.158485151112061
Joints:
- removed joint laser_joint
- joint left_wheel_joint: origin xyz=0.2435 0 0.06725 rpy=-1.5533 0.017448 -1.5705 -> xyz=0 0.239998 0.0392500000000001 rpy=1.5707963267949 0 3.14159265358979
- joint right_wheel_joint: origin xyz=-0.2435 0 0.06725 rpy=1.5708 0 -1.5708 -> xyz=0 -0.239998 0.03925 rpy=1.5707963267949 0 0

Commit message: adding changes

File: slam/delivery_robot/urdf/delivery_robot.urdf (robot description, URDF)
Before this commit: robot delivery_robot, 3 links, 2 joints
Links:
- added link laser, mass 0.114; collision cylinder length=0.0315 radius=0.055; visual mesh filename=package://delivery_robot/meshes/lds.stl scale=0.001 0.001 0.001
- link base_link: mass 3.92914679746778 -> 5.1663
- link left_wheel: mass 0.158485151112061 -> 0.15849
- link right_wheel: mass 0.158485151112061 -> 0.15849
Joints:
- added joint laser_joint: type fixed, parent base_link, child laser, origin xyz=0.0 0 0.244 rpy=0 0 0, axis 0 1 0
- joint left_wheel_joint: origin xyz=0 0.239998 0.0392500000000001 rpy=1.5707963267949 0 3.14159265358979 -> xyz=0.2435 0 0.06725 rpy=-1.5533 0.017448 -1.5705
- joint right_wheel_joint: origin xyz=0 -0.239998 0.03925 rpy=1.5707963267949 0 0 -> xyz=-0.2435 0 0.06725 rpy=1.5708 0 -1.5708
