Commit message: add laser_scan to delivery_robot_urdf2

File: slam/delivery_robot_urdf2/urdf/delivery_robot_urdf2.urdf (robot description, URDF)
Before this commit: robot delivery_robot_urdf2, 3 links, 2 joints
Links:
- added link laser, mass 0.114; collision cylinder length=0.0315 radius=0.055; visual mesh filename=package://delivery_robot_urdf2/meshes/lds.stl scale=0.001 0.001 0.001
Joints:
- added joint laser_joint: type fixed, parent base_link, child laser, origin xyz=0.0 0 0.244 rpy=0 0 0, axis 0 1 0

Commit message: add base_footprint to the robot urdf

File: slam/delivery_robot_urdf2/urdf/delivery_robot_urdf2.urdf (robot description, URDF)
Before this commit: robot delivery_robot_urdf2, 4 links, 3 joints
Links:
- added link base_footprint
Joints:
- added joint base_footprint_joint: type fixed, parent base_footprint, child base_link, origin xyz=0 0 0 rpy=0 0 0

Commit message: add ekf to amcl

File: slam/delivery_robot_urdf2/urdf/delivery_robot_urdf2.urdf (robot description, URDF)
Before this commit: robot delivery_robot_urdf2, 4 links, 3 joints
Links:
- added link base_footprint
- added link imu_link
Joints:
- added joint base_footprint_joint: type fixed, parent base_footprint, child base_link, origin xyz=0 0 0 rpy=0 0 0
- added joint imu_joint: type fixed, parent base_link, child imu_link, origin xyz=0 0 0.1 rpy=0 0 0
